File: Hardware/ADC_voltage_dividers.sch (KiCad schematic (older format))
At the start: 5 parts

Commit message: associated components to their JLC part numbers
Parts:
- R29: LCSC (none) -> C22813
- R30: LCSC (none) -> C25950
- R32, R33: LCSC (none) -> C31850
Changed lines of the file:
@@
 EESchema Schematic File Version 4
-LIBS:ZP-Breakout-cache
-EELAYER 29 0
+EELAYER 30 0
 EELAYER END
 $Descr A4 11693 8268
@@
 F 3 "http://www.yageo.com/documents/recent/PYu-RC_Group_51_RoHS_L_10.pdf" H 3850 2900 50  0001 C CNN
 F 4 "RESS-002" V 3850 2900 60  0001 C CNN "part_num"
+F 5 " C31850" V 3850 2900 50  0001 C CNN "LCSC"
 	1    3850 2900
 	1    0    0    -1
@@
 F 3 "http://www.yageo.com/documents/recent/PYu-RC_Group_51_RoHS_L_10.pdf" H 3400 2700 50  0001 C CNN
 F 4 "RESS-007" V 3400 2700 60  0001 C CNN "part_num"
+F 5 "C22813" V 3400 2700 50  0001 C CNN "LCSC"
 	1    3400 2700
 	0    1    1    0
@@
 F 3 "http://www.yageo.com/documents/recent/PYu-RC_Group_51_RoHS_L_10.pdf" H 3850 3900 50  0001 C CNN
 F 4 "RESS-002" V 3850 3900 60  0001 C CNN "part_num"
+F 5 "C31850" V 3850 3900 50  0001 C CNN "LCSC"
 	1    3850 3900
 	1    0    0    -1
@@
 F 3 "http://www.yageo.com/documents/recent/PYu-RC_Group_51_RoHS_L_10.pdf" H 3450 3600 50  0001 C CNN
 F 4 "RESS-004" V 3450 3600 60  0001 C CNN "part_num"
+F 5 "C25950" V 3450 3600 50  0001 C CNN "LCSC"
 	1    3450 3600
 	0    1    1    0
