File: Hardware/HEADERS.sch (KiCad schematic (older format))
At the start: 51 parts, among them J10 GH-4, J11 GH-3, J12 GH-4, J13 GH-2, J14 GH-4, J15 GH-4, J16 GH-4, J17 GH-4, J18 GH-6, J19 GH-6, J20 GH-6, J21 GH-6, J22 GH-6, J23 GH-6, J24 GH-2, J25 GH-4, J26 GH-4, J27 GH-4, J28 GH-4, J29 GH-6, J7 GH-2, Q1 BSS84LT1G, Q3 BSS84LT1G, SW1 SW_Push_Dual_1-2short_3-4short, SW2 SW_Push_Dual_1-2short_3-4short

Commit message: Finished routing. TODO: Silk.
Parts:
- J27: value GH-4 -> GH-2; footprint Connector_PinHeader_2.54mm:PinHeader_1x04_P2.54mm_Vertical -> Connector_PinHeader_2.54mm:PinHeader_1x02_P2.54mm_Vertical; symbol Connector_Generic:Conn_01x04 -> Connector_Generic:Conn_01x02
Connections:
- net GND: no longer J27.1 (Pin_1)
- net I2C_PULLUP: now also Q1.2 (D), Q3.2 (D), R1.2, R2.2
- net SCL1: now also J27.1 (Pin_1); no longer J27.2 (Pin_2)
- net SDA1: now also J27.2 (Pin_2); no longer J27.3 (Pin_3)
- net V_I2C: no longer J27.4 (Pin_4), Q1.2 (D), Q3.2 (D), R1.2, R2.2
Other:
- note added: "Note: I2C_PULLUP is 3V3_INT\n"
- note removed: "Note: V_I2C is 3V3_INT\n"
Changed lines of the file:
@@
 Connection ~ 4050 4500
-Wire Wire Line
-	4200 2000 4200 2350
 Wire Wire Line
 	3900 3800 3950 3800
@@
 NRST_SAFETY
 Connection ~ 9650 5100
-Text HLabel 9300 2250 0    60   Input ~ 0
-V_I2C
 Wire Wire Line
 	9350 2250 9300 2250
@@
 	9350 2250 9350 2700
 Text Notes 9350 1750 0    60   ~ 0
-Note: V_I2C is 3V3_INT\n
+Note: I2C_PULLUP is 3V3_INT\n
 Wire Wire Line
 	9700 5950 9700 6150
@@
 	10550 2900 10550 3000
 Connection ~ 9700 5950
-Text HLabel 10500 2050 0    60   Input ~ 0
-V_I2C
 Wire Wire Line
 	10550 2050 10500 2050
@@
 Wire Wire Line
 	3900 3150 4500 3150
-Wire Wire Line
-	3900 2650 4050 2650
-Wire Wire Line
-	4050 2650 4050 3250
 Connection ~ 4050 3900
 Wire Wire Line
 	3900 3250 4050 3250
-Connection ~ 4050 3250
 Wire Wire Line
 	4050 3250 4050 3900
-Wire Wire Line
-	3900 2350 4200 2350
-Connection ~ 4200 2350
-Wire Wire Line
-	4200 2350 4200 2950
 Wire Wire Line
 	3900 2950 4200 2950
@@
 $EndComp
 $Comp
-L Connector_Generic:Conn_01x04 J27
+L Connector_Generic:Conn_01x02 J27
 U 1 1 604C5194
 P 3700 2550
 F 0 "J27" H 3800 2800 60  0000 C CNN
-F 1 "GH-4" H 3800 2300 60  0000 C CNN
-F 2 "Connector_PinHeader_2.54mm:PinHeader_1x04_P2.54mm_Vertical" H 3700 2600 60  0001 C CNN
+F 1 "GH-2" H 3800 2300 60  0000 C CNN
+F 2 "Connector_PinHeader_2.54mm:PinHeader_1x02_P2.54mm_Vertical" H 3700 2600 60  0001 C CNN
 F 3 "http://www.jst-mfg.com/product/pdf/eng/eGH.pdf" H 3700 2600 60  0001 C CNN
 F 4 "CONN-08" H 3900 2900 60  0001 C CNN "part_num"
@@
 Wire Wire Line
 	9250 5450 9200 5450
-Text HLabel 9150 4300 0    60   Input ~ 0
-V_I2C
-Text HLabel 9200 5450 0    60   Input ~ 0
-V_I2C
 Wire Wire Line
 	10800 5950 10800 6300
@@
 	8050 3000 8050 3850
 Connection ~ 8050 3850
+Wire Wire Line
+	4200 2000 4200 2950
+Text HLabel 9300 2250 0    60   Input ~ 0
+I2C_PULLUP
+Text HLabel 10500 2050 0    60   Input ~ 0
+I2C_PULLUP
+Text HLabel 9150 4300 0    60   Input ~ 0
+I2C_PULLUP
+Text HLabel 9200 5450 0    60   Input ~ 0
+I2C_PULLUP
 $EndSCHEMATC

Commit message: Added additional headers to some interfaces, GPIOs, and FTDI pins. Added silks
Parts:
- removed TP19: TDO1_TST, TestPoint:TestPoint_Pad_D1.5mm, symbol Connector:TestPoint
- removed TP20: TMS1_TST, TestPoint:TestPoint_Pad_D1.5mm, symbol Connector:TestPoint
- removed TP21: TDO2_TST, TestPoint:TestPoint_Pad_D1.5mm, symbol Connector:TestPoint
- removed TP22: TMS2_TST, TestPoint:TestPoint_Pad_D1.5mm, symbol Connector:TestPoint
- removed TP23: UART1_RTS_TST, TestPoint:TestPoint_Pad_D1.5mm, symbol Connector:TestPoint
- removed TP24: UART1_CTS_TST, TestPoint:TestPoint_Pad_D1.5mm, symbol Connector:TestPoint
- removed TP25: UART2_RTS_TST, TestPoint:TestPoint_Pad_D1.5mm, symbol Connector:TestPoint
- removed TP26: UART2_CTS_TST, TestPoint:TestPoint_Pad_D1.5mm, symbol Connector:TestPoint
- added J1, TMS1: GH-4, Connector_PinHeader_2.54mm:PinHeader_1x04_P2.54mm_Vertical, symbol Connector_Generic:Conn_01x04
- added PPM1: GH-3, Connector_PinHeader_2.54mm:PinHeader_1x03_P2.54mm_Vertical, symbol Connector_Generic:Conn_01x03
- added SPI6_SAFE_AUTO1: GH-6, Connector_PinHeader_2.54mm:PinHeader_1x06_P2.54mm_Vertical, symbol Connector_Generic:Conn_01x06
- AIRSPEED1: renamed from J11; part_num CONN-07 -> CONN-007
- GPIO_AUTO1: renamed from J15; part_num CONN-08 -> CONN-008
- GPIO_SAFE1: renamed from J16; part_num CONN-08 -> CONN-008
- I2C1_SAFE_AUTO1: renamed from J27; part_num CONN-08 -> CONN-008
- I2C2_ALT1: renamed from J28; part_num CONN-08 -> CONN-008
- I2C4: renamed from J17; part_num CONN-08 -> CONN-008
- RSSI1: renamed from J10; value GH-4 -> GH-3; footprint Connector_PinHeader_2.54mm:PinHeader_1x04_P2.54mm_Vertical -> Connector_PinHeader_2.54mm:PinHeader_1x03_P2.54mm_Vertical; symbol Connector_Generic:Conn_01x04 -> Connector_Generic:Conn_01x03; part_num CONN-08 -> CONN-009
- SPI1_IMU1: renamed from J29; part_num CONN-09 -> CONN-009
- SPI2: renamed from J21; part_num CONN-09 -> CONN-009
- SPI4: renamed from J22; part_num CONN-09 -> CONN-009
- SPI5: renamed from J23; part_num CONN-09 -> CONN-009
- SWD_AUTO1: renamed from J26; part_num CONN-08 -> CONN-009
- SWD_SAFE1: renamed from J25; part_num CONN-08 -> CONN-009
- UART1: renamed from J18; part_num CONN-09 -> CONN-009
- UART2: renamed from J20; part_num CONN-09 -> CONN-009
- UART4: renamed from J19; part_num CONN-09 -> CONN-009
- UART_DBG_AUTO1: renamed from J24; part_num CONN-06 -> CONN-006
- UART_DBG_SAFE1: renamed from J7; part_num CONN-06 -> CONN-006
- UHF1: renamed from J14; part_num CONN-08 -> CONN-008
- USS1: renamed from J12; part_num CONN-08 -> CONN-008
- V_ISNS1: renamed from J13; part_num CONN-06 -> CONN-006
Connections:
- net GND: now also PPM1.1 (Pin_1), SPI6_SAFE_AUTO1.1 (Pin_1); no longer GPIO_AUTO1.1 (Pin_1)
- net PPM: now also PPM1.3 (Pin_3); no longer RSSI1.3 (Pin_3)
- net RSSI: now also RSSI1.3 (Pin_3); no longer RSSI1.2 (Pin_2)
- net SCL4: no longer GPIO_AUTO1.2 (Pin_2), GPIO_SAFE1.2 (Pin_2)
- net SDA4: no longer GPIO_AUTO1.3 (Pin_3), GPIO_SAFE1.3 (Pin_3)
- net TDO1_TST: now also TMS1.4 (Pin_4)
- net TDO2_TST: now also TMS1.2 (Pin_2)
- net TMS1_TST: now also TMS1.3 (Pin_3)
- net TMS2_TST: now also TMS1.1 (Pin_1)
- net UART1_CTS_TST: now also J1.3 (Pin_3)
- net UART1_RTS_TST: now also J1.4 (Pin_4)
- net UART2_CTS_TST: now also J1.1 (Pin_1)
- net UART2_RTS_TST: now also J1.2 (Pin_2)
- net V_I2C: no longer GPIO_AUTO1.4 (Pin_4), GPIO_SAFE1.4 (Pin_4)
- net V_SPI: now also SPI6_SAFE_AUTO1.6 (Pin_6)
- removed net V_PPM: RSSI1.4 (Pin_4)
- new net PB1: GPIO_AUTO1.2 (Pin_2)
- new net PB2: GPIO_AUTO1.1 (Pin_1)
- new net PC4: GPIO_AUTO1.4 (Pin_4)
- new net PC5: GPIO_AUTO1.3 (Pin_3)
- new net SPI6_CK: SPI6_SAFE_AUTO1.5 (Pin_5)
- new net SPI6_SDO: SPI6_SAFE_AUTO1.4 (Pin_4)
- new net SPI6_SI: SPI6_SAFE_AUTO1.3 (Pin_3)
- new net SPI6_SS: SPI6_SAFE_AUTO1.2 (Pin_2)
- new net S_PC12: GPIO_SAFE1.2 (Pin_2)
- new net S_PC2: GPIO_SAFE1.3 (Pin_3)
- new net S_PC3: GPIO_SAFE1.4 (Pin_4)
- no-connect marks 0 -> 2
Other:
- moved on the sheet: AIRSPEED1, GPIO_AUTO1, GPIO_SAFE1, UART_DBG_AUTO1, UART_DBG_SAFE1, UHF1, USS1, V_ISNS1

Commit message: associated components to their JLC part numbers
Parts:
- C8, C9: LCSC (none) -> C14663
- D2, D3: LCSC (none) -> C72043
- R1, R2, R44, R45, R46, R47, R48, R49: LCSC (none) -> C25804
- R3, R4: LCSC (none) -> C22775
- SW1, SW2: symbol WARG:SW_Push_Dual_1-2short_3-4short -> ZP-Breakout-rescue:SW_Push_Dual_1-2short_3-4short-WARG
Changed lines of the file:
@@
 EESchema Schematic File Version 4
-LIBS:ZP-Breakout-cache
-EELAYER 29 0
+EELAYER 30 0
 EELAYER END
 $Descr A4 11693 8268
@@
 $EndComp
 $Comp
-L WARG:SW_Push_Dual_1-2short_3-4short SW?
+L ZP-Breakout-rescue:SW_Push_Dual_1-2short_3-4short-WARG SW?
 U 1 1 602F1065
 P 10000 5100
@@
 F 3 "http://www.yageo.com/documents/recent/PYu-RC_Group_51_RoHS_L_10.pdf" H 9250 4700 50  0001 C CNN
 F 4 "RESS-005" V 9250 4700 60  0001 C CNN "part_num"
+F 5 " C25804" V 9250 4700 50  0001 C CNN "LCSC"
 	1    9250 4700
 	-1   0    0    1
@@
 F 3 "http://optoelectronics.liteon.com/upload/download/DS22-2000-228/LTST-C191KGKT.PDF" H 9350 3350 50  0001 C CNN
 F 4 "DIOD-002" H 9350 3350 60  0001 C CNN "part_num"
+F 5 "C72043" H 9350 3350 50  0001 C CNN "LCSC"
 	1    9350 3350
 	0    -1   -1   0
@@
 F 3 "http://www.yageo.com/documents/recent/PYu-RC_Group_51_RoHS_L_10.pdf" H 9350 3700 50  0001 C CNN
 F 4 "RESS-006" V 9350 3700 60  0001 C CNN "part_num"
+F 5 "C22775" V 9350 3700 50  0001 C CNN "LCSC"
 	1    9350 3700
 	1    0    0    -1
@@
 $EndComp
 $Comp
-L WARG:SW_Push_Dual_1-2short_3-4short SW?
+L ZP-Breakout-rescue:SW_Push_Dual_1-2short_3-4short-WARG SW?
 U 1 1 6035554F
 P 10050 5950
@@
 F 3 "http://optoelectronics.liteon.com/upload/download/DS22-2000-228/LTST-C191KGKT.PDF" H 10550 3150 50  0001 C CNN
 F 4 "DIOD-002" H 10550 3150 60  0001 C CNN "part_num"
+F 5 "C72043" H 10550 3150 50  0001 C CNN "LCSC"
 	1    10550 3150
 	0    -1   -1   0
@@
 F 3 "http://www.yageo.com/documents/recent/PYu-RC_Group_51_RoHS_L_10.pdf" H 10550 3500 50  0001 C CNN
 F 4 "RESS-006" V 10550 3500 60  0001 C CNN "part_num"
+F 5 "C22775" V 10550 3500 50  0001 C CNN "LCSC"
 	1    10550 3500
 	1    0    0    -1
@@
 F 3 "http://industrial.panasonic.com/www-cgi/jvcr13pz.cgi?E+PZ+3+AOA0001+ERJ3GEYJ103V+7+WW" H 2700 1250 50  0001 C CNN
 F 4 "RESS-005" V 2700 1250 60  0001 C CNN "part_num"
+F 5 " C25804" V 2700 1250 50  0001 C CNN "LCSC"
 	1    2700 1250
 	1    0    0    -1
@@
 F 3 "http://industrial.panasonic.com/www-cgi/jvcr13pz.cgi?E+PZ+3+AOA0001+ERJ3GEYJ103V+7+WW" H 2900 1250 50  0001 C CNN
 F 4 "RESS-005" V 2900 1250 60  0001 C CNN "part_num"
+F 5 " C25804" V 2900 1250 50  0001 C CNN "LCSC"
 	1    2900 1250
 	1    0    0    -1
@@
 F 3 "http://industrial.panasonic.com/www-cgi/jvcr13pz.cgi?E+PZ+3+AOA0001+ERJ3GEYJ103V+7+WW" H 4050 1250 50  0001 C CNN
 F 4 "RESS-005" V 4050 1250 60  0001 C CNN "part_num"
+F 5 " C25804" V 4050 1250 50  0001 C CNN "LCSC"
 	1    4050 1250
 	1    0    0    -1
@@
 F 3 "http://industrial.panasonic.com/www-cgi/jvcr13pz.cgi?E+PZ+3+AOA0001+ERJ3GEYJ103V+7+WW" H 4250 1250 50  0001 C CNN
 F 4 "RESS-005" V 4250 1250 60  0001 C CNN "part_num"
+F 5 " C25804" V 4250 1250 50  0001 C CNN "LCSC"
 	1    4250 1250
 	1    0    0    -1
@@
 F 3 "http://industrial.panasonic.com/www-cgi/jvcr13pz.cgi?E+PZ+3+AOA0001+ERJ3GEYJ103V+7+WW" H 3600 1250 50  0001 C CNN
 F 4 "RESS-005" V 3600 1250 60  0001 C CNN "part_num"
+F 5 " C25804" V 3600 1250 50  0001 C CNN "LCSC"
 	1    3600 1250
 	1    0    0    -1
@@
 F 3 "http://industrial.panasonic.com/www-cgi/jvcr13pz.cgi?E+PZ+3+AOA0001+ERJ3GEYJ103V+7+WW" H 3400 1250 50  0001 C CNN
 F 4 "RESS-005" V 3400 1250 60  0001 C CNN "part_num"
+F 5 " C25804" V 3400 1250 50  0001 C CNN "LCSC"
 	1    3400 1250
 	1    0    0    -1
@@
 F 3 "http://www.yageo.com/documents/recent/PYu-RC_Group_51_RoHS_L_10.pdf" H 9250 5650 50  0001 C CNN
 F 4 "RESS-005" V 9250 5650 60  0001 C CNN "part_num"
+F 5 "C25804" V 9250 5650 50  0001 C CNN "LCSC"
 	1    9250 5650
 	-1   0    0    1
@@
 F 3 "https://search.murata.co.jp/Ceramy/image/img/A01X/G101/ENG/GRM188R71E104KA01-01.pdf" H 9400 5300 50  0001 C CNN
 F 4 "CAPP-005" H 9400 5300 60  0001 C CNN "part_num"
+F 5 "C14663" H 9400 5300 50  0001 C CNN "LCSC"
 	1    9400 5300
 	1    0    0    -1
@@
 F 3 "https://search.murata.co.jp/Ceramy/image/img/A01X/G101/ENG/GRM188R71E104KA01-01.pdf" H 9350 6150 50  0001 C CNN
 F 4 "CAPP-005" H 9350 6150 60  0001 C CNN "part_num"
+F 5 "C14663" H 9350 6150 50  0001 C CNN "LCSC"
 	1    9350 6150
 	1    0    0    -1
