File: Hardware/POWER.sch (KiCad schematic (older format))
At the start: 17 parts, among them J30 Conn_02x02_Odd_Even, J31 Conn_01x02, U1 MCP1826S-3302E/DB

Commit message: Finished routing. TODO: Silk.
Connections:
- net 5V_INT: now also J30.4 (Pin_4); no longer J30.2 (Pin_2)
- net 6V_EXT: now also J30.2 (Pin_2); no longer J30.4 (Pin_4)
Other:
- moved on the sheet: D16, R8, R9
Changed lines of the file:
@@
 Text HLabel 6600 2900 0    60   Input ~ 0
 5V_USB+
-Wire Wire Line
-	9450 2900 10250 2900
-Text HLabel 10250 2900 2    60   Output ~ 0
+Text HLabel 10500 3000 2    60   Output ~ 0
 6V_EXT
-Text Label 9500 2900 0    60   ~ 0
+Text Label 9500 3000 0    60   ~ 0
 6V_EXT
 Connection ~ 9000 5650
@@
 Text HLabel 9800 3100 2    60   Output ~ 0
 3V3
-Text Label 9500 3000 0    59   ~ 0
+Text Label 9500 2900 0    59   ~ 0
 5V_INT
-Wire Wire Line
-	10300 3000 10500 3000
-Connection ~ 10300 3000
-Wire Wire Line
-	10300 3000 10300 3250
-Wire Wire Line
-	9450 3000 10300 3000
 $Comp
 L Device:R R8
 U 1 1 5CC233BF
-P 10300 3400
-F 0 "R8" V 10380 3400 50  0000 C CNN
-F 1 "100" V 10300 3400 50  0000 C CNN
-F 2 "Resistor_SMD:R_0603_1608Metric_Pad0.84x1.00mm_HandSolder" V 10230 3400 50  0001 C CNN
-F 3 "http://www.yageo.com/documents/recent/PYu-RC_Group_51_RoHS_L_10.pdf" H 10300 3400 50  0001 C CNN
-F 4 "RESS-006" V 10300 3400 60  0001 C CNN "part_num"
-	1    10300 3400
+P 10100 3350
+F 0 "R8" V 10180 3350 50  0000 C CNN
+F 1 "100" V 10100 3350 50  0000 C CNN
+F 2 "Resistor_SMD:R_0603_1608Metric_Pad0.84x1.00mm_HandSolder" V 10030 3350 50  0001 C CNN
+F 3 "http://www.yageo.com/documents/recent/PYu-RC_Group_51_RoHS_L_10.pdf" H 10100 3350 50  0001 C CNN
+F 4 "RESS-006" V 10100 3350 60  0001 C CNN "part_num"
+	1    10100 3350
 	1    0    0    -1
 $EndComp
@@
 L power:GND #PWR0108
 U 1 1 5CC21AE8
-P 10300 4300
-F 0 "#PWR0108" H 10300 4050 50  0001 C CNN
-F 1 "GND" H 10300 4150 50  0000 C CNN
-F 2 "" H 10300 4300 50  0000 C CNN
-F 3 "" H 10300 4300 50  0000 C CNN
-	1    10300 4300
-	1    0    0    -1
-$EndComp
-Wire Wire Line
-	10300 3850 10300 4000
+P 10100 4250
+F 0 "#PWR0108" H 10100 4000 50  0001 C CNN
+F 1 "GND" H 10100 4100 50  0000 C CNN
+F 2 "" H 10100 4250 50  0000 C CNN
+F 3 "" H 10100 4250 50  0000 C CNN
+	1    10100 4250
+	1    0    0    -1
+$EndComp
+Wire Wire Line
+	10100 3800 10100 3950
 $Comp
 L Device:R R9
 U 1 1 5CBD97C2
-P 10300 3700
-F 0 "R9" V 10380 3700 50  0000 C CNN
-F 1 "100" V 10300 3700 50  0000 C CNN
-F 2 "Resistor_SMD:R_0603_1608Metric_Pad0.84x1.00mm_HandSolder" V 10230 3700 50  0001 C CNN
-F 3 "http://www.yageo.com/documents/recent/PYu-RC_Group_51_RoHS_L_10.pdf" H 10300 3700 50  0001 C CNN
-F 4 "RESS-006" V 10300 3700 60  0001 C CNN "part_num"
-	1    10300 3700
+P 10100 3650
+F 0 "R9" V 10180 3650 50  0000 C CNN
+F 1 "100" V 10100 3650 50  0000 C CNN
+F 2 "Resistor_SMD:R_0603_1608Metric_Pad0.84x1.00mm_HandSolder" V 10030 3650 50  0001 C CNN
+F 3 "http://www.yageo.com/documents/recent/PYu-RC_Group_51_RoHS_L_10.pdf" H 10100 3650 50  0001 C CNN
+F 4 "RESS-006" V 10100 3650 60  0001 C CNN "part_num"
+	1    10100 3650
 	1    0    0    -1
 $EndComp
@@
 L Device:LED D16
 U 1 1 5CBD935A
-P 10300 4150
-F 0 "D16" H 10300 4250 50  0000 C CNN
-F 1 "PWR_LED" H 10300 4050 50  0000 C CNN
-F 2 "LED_SMD:LED_0603_1608Metric_Pad0.67x1.00mm_HandSolder" H 10300 4150 50  0001 C CNN
-F 3 "http://optoelectronics.liteon.com/upload/download/DS22-2000-223/LTST-C191KRKT.PDF" H 10300 4150 50  0001 C CNN
-F 4 "DIOD-003" H 10300 4150 60  0001 C CNN "part_num"
-	1    10300 4150
+P 10100 4100
+F 0 "D16" H 10100 4200 50  0000 C CNN
+F 1 "PWR_LED" H 10100 4000 50  0000 C CNN
+F 2 "LED_SMD:LED_0603_1608Metric_Pad0.67x1.00mm_HandSolder" H 10100 4100 50  0001 C CNN
+F 3 "http://optoelectronics.liteon.com/upload/download/DS22-2000-223/LTST-C191KRKT.PDF" H 10100 4100 50  0001 C CNN
+F 4 "DIOD-003" H 10100 4100 60  0001 C CNN "part_num"
+	1    10100 4100
 	0    1    -1   0
 $EndComp
-Text HLabel 10500 3000 2    60   Output ~ 0
+Text HLabel 10250 2900 2    60   Output ~ 0
 5V_INT
 Wire Wire Line
@@
 Wire Wire Line
 	9250 3100 9600 3100
+Wire Wire Line
+	9450 3000 10500 3000
+Wire Wire Line
+	10100 3200 10100 2900
+Wire Wire Line
+	9450 2900 10100 2900
+Connection ~ 10100 2900
+Wire Wire Line
+	10100 2900 10250 2900
 $EndSCHEMATC

Commit message: associated components to their JLC part numbers
Parts:
- C1, C2: LCSC (none) -> C57112
- C3, C4: LCSC (none) -> C19666
- C5, C6: LCSC (none) -> C15849
- C7: LCSC (none) -> C14663
- D15, D16: LCSC (none) -> C2286
- R7, R8, R9: LCSC (none) -> C22775
- U1: LCSC (none) -> C6186
Changed lines of the file:
@@
 EESchema Schematic File Version 4
-LIBS:ZP-Breakout-cache
-EELAYER 29 0
+EELAYER 30 0
 EELAYER END
 $Descr A4 11693 8268
@@
 F 3 "https://search.murata.co.jp/Ceramy/image/img/A01X/G101/ENG/GRM188R61E105KA12-01.pdf" H 10050 5400 50  0001 C CNN
 F 4 "CAPP-004" H 10050 5400 60  0001 C CNN "part_num"
+F 5 "C15849" H 10050 5400 50  0001 C CNN "LCSC"
 	1    10050 5400
 	1    0    0    -1
@@
 F 3 "https://search.murata.co.jp/Ceramy/image/img/A01X/G101/ENG/GRM188R71E104KA01-01.pdf" H 10250 5400 50  0001 C CNN
 F 4 "CAPP-005" H 10250 5400 60  0001 C CNN "part_num"
+F 5 "C14663" H 10250 5400 50  0001 C CNN "LCSC"
 	1    10250 5400
 	1    0    0    -1
@@
 F 3 "http://ww1.microchip.com/downloads/en/DeviceDoc/22057B.pdf" H 9500 5750 60  0001 C CNN
 F 4 "REGU-002" H 9600 5850 60  0001 C CNN "part_num"
+F 5 "C6186" H 9550 5350 50  0001 C CNN "LCSC"
 	1    9550 5350
 	1    0    0    -1
@@
 F 3 "https://search.murata.co.jp/Ceramy/image/img/A01X/G101/ENG/GRM188R61E105KA12-01.pdf" H 8800 5400 50  0001 C CNN
 F 4 "CAPP-004" H 8800 5400 60  0001 C CNN "part_num"
+F 5 "C15849" H 8800 5400 50  0001 C CNN "LCSC"
 	1    8800 5400
 	1    0    0    -1
@@
 F 3 "https://search.murata.co.jp/Ceramy/image/img/A01X/G101/ENG/GRM188R71H103KA01-01.pdf" H 6800 3100 50  0001 C CNN
 F 4 "CAPP-010" H 6800 3100 60  0001 C CNN "part_num"
+F 5 "C57112" H 6800 3100 50  0001 C CNN "LCSC"
 	1    6800 3100
 	-1   0    0    1
@@
 F 3 "https://search.murata.co.jp/Ceramy/image/img/A01X/G101/ENG/GRM188R71H103KA01-01.pdf" H 7550 3100 50  0001 C CNN
 F 4 "CAPP-010" H 7550 3100 60  0001 C CNN "part_num"
+F 5 "C57112" H 7550 3100 50  0001 C CNN "LCSC"
 	1    7550 3100
 	-1   0    0    1
@@
 F 3 "http://www.samsungsem.com/kr/support/product-search/mlcc/CL10A475MP5LNNC.jsp" H 7850 3100 50  0001 C CNN
 F 4 "CAPP-006" H 7850 3100 60  0001 C CNN "part_num"
+F 5 "C19666" H 7850 3100 50  0001 C CNN "LCSC"
 	1    7850 3100
 	1    0    0    1
@@
 F 3 "http://www.samsungsem.com/kr/support/product-search/mlcc/CL10A475MP5LNNC.jsp" H 8400 5400 50  0001 C CNN
 F 4 "CAPP-006" H 8400 5400 60  0001 C CNN "part_num"
+F 5 "C19666" H 8400 5400 50  0001 C CNN "LCSC"
 	1    8400 5400
 	1    0    0    1
@@
 	8400 5200 8800 5200
 Connection ~ 8800 5200
-Wire Wire Line
-	8400 5200 8000 5200
-Connection ~ 8400 5200
 $Comp
 L Device:D D8
@@
 F 3 "http://www.yageo.com/documents/recent/PYu-RC_Group_51_RoHS_L_10.pdf" H 9600 3650 50  0001 C CNN
 F 4 "RESS-006" V 9600 3650 60  0001 C CNN "part_num"
+F 5 "C22775" V 9600 3650 50  0001 C CNN "LCSC"
 	1    9600 3650
 	1    0    0    -1
@@
 F 3 "http://optoelectronics.liteon.com/upload/download/DS22-2000-223/LTST-C191KRKT.PDF" H 9600 3950 50  0001 C CNN
 F 4 "DIOD-003" H 9600 3950 60  0001 C CNN "part_num"
+F 5 "C2286" H 9600 3950 50  0001 C CNN "LCSC"
 	1    9600 3950
 	0    -1   -1   0
@@
 F 3 "http://www.yageo.com/documents/recent/PYu-RC_Group_51_RoHS_L_10.pdf" H 10100 3350 50  0001 C CNN
 F 4 "RESS-006" V 10100 3350 60  0001 C CNN "part_num"
+F 5 "C22775" V 10100 3350 50  0001 C CNN "LCSC"
 	1    10100 3350
 	1    0    0    -1
@@
 F 3 "http://www.yageo.com/documents/recent/PYu-RC_Group_51_RoHS_L_10.pdf" H 10100 3650 50  0001 C CNN
 F 4 "RESS-006" V 10100 3650 60  0001 C CNN "part_num"
+F 5 "C22775" V 10100 3650 50  0001 C CNN "LCSC"
 	1    10100 3650
 	1    0    0    -1
@@
 F 3 "http://optoelectronics.liteon.com/upload/download/DS22-2000-223/LTST-C191KRKT.PDF" H 10100 4100 50  0001 C CNN
 F 4 "DIOD-003" H 10100 4100 60  0001 C CNN "part_num"
+F 5 "C2286" H 10100 4100 50  0001 C CNN "LCSC"
 	1    10100 4100
 	0    1    -1   0
