File: Hardware/SENSORS.sch (KiCad schematic (older format))
At the start: 7 parts, among them U6 ICM-20602, U7 MS5637-02BA03

Commit message: associated components to their JLC part numbers
Parts:
- C43: LCSC (none) -> C57112
- C44, C46, C47: LCSC (none) -> C14663
- C45: LCSC (none) -> C23630
- U6: symbol WARG:ICM-20602 -> ZP-Breakout-rescue:ICM-20602-WARG
- U7: symbol WARG:MS5637-02BA03 -> ZP-Breakout-rescue:MS5637-02BA03-WARG
Changed lines of the file:
@@
 EESchema Schematic File Version 4
-LIBS:ZP-Breakout-cache
-EELAYER 29 0
+EELAYER 30 0
 EELAYER END
 $Descr A4 11693 8268
@@
 Connection ~ 2700 2800
 $Comp
-L WARG:MS5637-02BA03 U7
+L ZP-Breakout-rescue:MS5637-02BA03-WARG U7
 U 1 1 5B0F962E
 P 6200 3650
@@
 F 3 "https://search.murata.co.jp/Ceramy/image/img/A01X/G101/ENG/GRM188R71E104KA01-01.pdf" H 6200 3050 50  0001 C CNN
 F 4 "CAPP-005" H 6200 3050 60  0001 C CNN "part_num"
+F 5 "C14663" H 6200 3050 50  0001 C CNN "LCSC"
 	1    6200 3050
 	0    1    1    0
@@
 F 3 "https://search.murata.co.jp/Ceramy/image/img/A01X/G101/ENG/GRM188R71E104KA01-01.pdf" H 3750 3050 50  0001 C CNN
 F 4 "CAPP-005" H 3750 3050 60  0001 C CNN "part_num"
+F 5 "C14663" H 3750 3050 50  0001 C CNN "LCSC"
 	1    3750 3050
 	1    0    0    -1
@@
 F 3 "https://ds.yuden.co.jp/TYCOMPAS/ut/specSheet?pn=TMK107ABJ225KA-T++" H 2700 2950 50  0001 C CNN
 F 4 "CAPP-007" H 2700 2950 60  0001 C CNN "part_num"
+F 5 "C23630" H 2700 2950 50  0001 C CNN "LCSC"
 	1    2700 2950
 	1    0    0    -1
@@
 F 3 "https://search.murata.co.jp/Ceramy/image/img/A01X/G101/ENG/GRM188R71E104KA01-01.pdf" H 2400 2950 50  0001 C CNN
 F 4 "CAPP-005" H 2400 2950 60  0001 C CNN "part_num"
+F 5 "C14663" H 2400 2950 50  0001 C CNN "LCSC"
 	1    2400 2950
 	1    0    0    -1
@@
 F 3 "https://search.murata.co.jp/Ceramy/image/img/A01X/G101/ENG/GRM188R71H103KA01-01.pdf" H 1700 3600 50  0001 C CNN
 F 4 "CAPP-010" H 1700 3600 60  0001 C CNN "part_num"
+F 5 "C57112" H 1700 3600 50  0001 C CNN "LCSC"
 	1    1700 3600
 	-1   0    0    1
 $EndComp
 $Comp
-L WARG:ICM-20602 U?
+L ZP-Breakout-rescue:ICM-20602-WARG U?
 U 1 1 5B0F92D3
 P 3150 3650
