File: Hardware/USB INTERFACE.sch (KiCad schematic (older format))
At the start: 35 parts, among them J9 USB_MICRO_B, U8 FT4232H, Y3 Crystal_GND24

Commit message: associated components to their JLC part numbers
Parts:
- C48, C49, C50, C51, C52, C53, C54, C55, C57, C58, C64: LCSC (none) -> C14663
- C56: LCSC (none) -> C51412
- C59, C60, C63: LCSC (none) -> C19666
- J9: symbol Connector:USB_B_Micro -> ZP-Breakout-rescue:USB_B_Micro-Connector
- R34: LCSC (none) -> C23162
- R35: LCSC (none) -> C25804
- R36: LCSC (none) -> C22790
- R37, R38: LCSC (none) -> C22859
- R39: LCSC (none) -> C21190
- R40, R43: LCSC (none) -> C22962
- R41, R42: LCSC (none) -> C21189
- U8: LCSC (none) -> C56742
Changed lines of the file:
@@
 EESchema Schematic File Version 4
-LIBS:ZP-Breakout-cache
-EELAYER 29 0
+EELAYER 30 0
 EELAYER END
 $Descr A4 11693 8268
@@
 F 3 "https://www.ftdichip.com/Support/Documents/DataSheets/ICs/DS_FT4232H.pdf" H 950 4800 60  0001 C CNN
 F 4 "CHIP-005" H 1550 5900 60  0000 C CNN "part_num"
+F 5 "C56742" H 1550 5150 50  0001 C CNN "LCSC"
 	3    1550 5150
 	1    0    0    -1
 $EndComp
 $Comp
-L Connector:USB_B_Micro J9
+L ZP-Breakout-rescue:USB_B_Micro-Connector J9
 U 1 1 5B18AAF8
 P 1200 1700
+AR Path="/5B18AAF8" Ref="J9"  Part="1"
+AR Path="/5B2B4997/5B18AAF8" Ref="J9"  Part="1"
 F 0 "J9" H 1150 2250 50  0000 L CNN
 F 1 "USB_MICRO_B" H 950 2400 50  0000 L CNN
@@
 F 3 "https://search.murata.co.jp/Ceramy/image/img/A01X/G101/ENG/GRM188R71E104KA01-01.pdf" H 2450 5350 50  0001 C CNN
 F 4 "CAPP-005" H 2450 5350 60  0001 C CNN "part_num"
+F 5 "C14663" H 2450 5350 50  0001 C CNN "LCSC"
 	1    2450 5350
 	1    0    0    -1
@@
 F 3 "http://www.samsungsem.com/kr/support/product-search/mlcc/CL10A475MP5LNNC.jsp" H 4950 5150 50  0001 C CNN
 F 4 "CAPP-006" H 4950 5150 60  0001 C CNN "part_num"
+F 5 "C19666" H 4950 5150 50  0001 C CNN "LCSC"
 	1    4950 5150
 	1    0    0    -1
@@
 F 3 "https://search.murata.co.jp/Ceramy/image/img/A01X/G101/ENG/GRM188R71E104KA01-01.pdf" H 2750 5350 50  0001 C CNN
 F 4 "CAPP-005" H 2750 5350 60  0001 C CNN "part_num"
+F 5 "C14663" H 2750 5350 50  0001 C CNN "LCSC"
 	1    2750 5350
 	1    0    0    -1
@@
 F 3 "https://search.murata.co.jp/Ceramy/image/img/A01X/G101/ENG/GRM188R71E104KA01-01.pdf" H 3050 5350 50  0001 C CNN
 F 4 "CAPP-005" H 3050 5350 60  0001 C CNN "part_num"
+F 5 "C14663" H 3050 5350 50  0001 C CNN "LCSC"
 	1    3050 5350
 	1    0    0    -1
@@
 F 3 "https://search.murata.co.jp/Ceramy/image/img/A01X/G101/ENG/GRM188R71E104KA01-01.pdf" H 1650 6150 50  0001 C CNN
 F 4 "CAPP-005" H 1650 6150 60  0001 C CNN "part_num"
+F 5 "C14663" H 1650 6150 50  0001 C CNN "LCSC"
 	1    1650 6150
 	1    0    0    -1
@@
 F 3 "https://search.murata.co.jp/Ceramy/image/img/A01X/G101/ENG/GRM188R71E104KA01-01.pdf" H 1950 6150 50  0001 C CNN
 F 4 "CAPP-005" H 1950 6150 60  0001 C CNN "part_num"
+F 5 "C14663" H 1950 6150 50  0001 C CNN "LCSC"
 	1    1950 6150
 	1    0    0    -1
@@
 F 3 "https://search.murata.co.jp/Ceramy/image/img/A01X/G101/ENG/GRM188R71E104KA01-01.pdf" H 2250 6150 50  0001 C CNN
 F 4 "CAPP-005" H 2250 6150 60  0001 C CNN "part_num"
+F 5 "C14663" H 2250 6150 50  0001 C CNN "LCSC"
 	1    2250 6150
 	1    0    0    -1
@@
 F 3 "http://www.samsungsem.com/kr/support/product-search/mlcc/CL10A475MP5LNNC.jsp" H 5250 5150 50  0001 C CNN
 F 4 "CAPP-006" H 5250 5150 60  0001 C CNN "part_num"
+F 5 "C19666" H 5250 5150 50  0001 C CNN "LCSC"
 	1    5250 5150
 	1    0    0    -1
@@
 F 3 "https://search.murata.co.jp/Ceramy/image/img/A01X/G101/ENG/GRM188R71E104KA01-01.pdf" H 4350 5150 50  0001 C CNN
 F 4 "CAPP-005" H 4350 5150 60  0001 C CNN "part_num"
+F 5 "C14663" H 4350 5150 50  0001 C CNN "LCSC"
 	1    4350 5150
 	1    0    0    -1
@@
 F 3 "https://search.murata.co.jp/Ceramy/image/img/A01X/G101/ENG/GRM188R71E104KA01-01.pdf" H 4650 5150 50  0001 C CNN
 F 4 "CAPP-005" H 4650 5150 60  0001 C CNN "part_num"
+F 5 "C14663" H 4650 5150 50  0001 C CNN "LCSC"
 	1    4650 5150
 	1    0    0    -1
@@
 F 3 "https://search.murata.co.jp/Ceramy/image/img/A01X/G101/ENG/GRM188R71E104KA01-01.pdf" H 6500 5150 50  0001 C CNN
 F 4 "CAPP-005" H 6500 5150 60  0001 C CNN "part_num"
+F 5 "C14663" H 6500 5150 50  0001 C CNN "LCSC"
 	1    6500 5150
 	1    0    0    -1
@@
 F 3 "http://www.samsungsem.com/kr/support/product-search/mlcc/CL10A475MP5LNNC.jsp" H 6200 5150 50  0001 C CNN
 F 4 "CAPP-006" H 6200 5150 60  0001 C CNN "part_num"
+F 5 "C19666" H 6200 5150 50  0001 C CNN "LCSC"
 	1    6200 5150
 	1    0    0    -1
@@
 F 3 "https://search.murata.co.jp/Ceramy/image/img/A01X/G101/ENG/GRM188R71E104KA01-01.pdf" H 2550 6150 50  0001 C CNN
 F 4 "CAPP-005" H 2550 6150 60  0001 C CNN "part_num"
+F 5 "C14663" H 2550 6150 50  0001 C CNN "LCSC"
 	1    2550 6150
 	1    0    0    -1
@@
 F 3 "https://search.murata.co.jp/Ceramy/image/img/A01X/G101/ENG/GRM188R71E104KA01-01.pdf" H 3500 5350 50  0001 C CNN
 F 4 "CAPP-005" H 3500 5350 60  0001 C CNN "part_num"
+F 5 "C14663" H 3500 5350 50  0001 C CNN "LCSC"
 	1    3500 5350
 	1    0    0    -1
@@
 F 3 "http://www.samsungsem.com/kr/support/product-search/mlcc/CL10A335KP8NNNC.jsp" H 3800 5350 50  0001 C CNN
 F 4 "CAPP-015" H 3800 5350 60  0001 C CNN "part_num"
+F 5 "C51412" H 3800 5350 50  0001 C CNN "LCSC"
 	1    3800 5350
 	1    0    0    -1
@@
 F 3 "http://www.yageo.com/NewPortal/yageodocoutput?fileName=/pdf/R-Chip/PYu-AC_51_RoHS_L_6.pdf" H 7950 1900 50  0001 C CNN
 F 4 "RESS-014" V 7950 1900 60  0001 C CNN "part_num"
+F 5 "C22962" V 7950 1900 50  0001 C CNN "LCSC"
 	1    7950 1900
 	0    1    1    0
@@
 F 3 "http://www.yageo.com/NewPortal/yageodocoutput?fileName=/pdf/R-Chip/PYu-AC_51_RoHS_L_6.pdf" H 9950 1900 50  0001 C CNN
 F 4 "RESS-014" V 9950 1900 60  0001 C CNN "part_num"
+F 5 "C22962" V 9950 1900 50  0001 C CNN "LCSC"
 	1    9950 1900
 	0    -1   1    0
@@
 F 3 "http://www.yageo.com/documents/recent/PYu-RC_Group_51_RoHS_L_10.pdf" H 9700 2000 50  0001 C CNN
 F 4 "RESS-001" V 9700 2000 60  0001 C CNN "part_num"
+F 5 "C21189" V 9700 2000 50  0001 C CNN "LCSC"
 	1    9700 2000
 	0    -1   1    0
@@
 F 3 "http://www.yageo.com/documents/recent/PYu-RC_Group_51_RoHS_L_10.pdf" H 8200 2000 50  0001 C CNN
 F 4 "RESS-001" V 8200 2000 60  0001 C CNN "part_num"
+F 5 "C21189" V 8200 2000 50  0001 C CNN "LCSC"
 	1    8200 2000
 	0    1    1    0
@@
 F 3 "http://www.yageo.com/NewPortal/yageodocoutput?fileName=/pdf/R-Chip/PYu-RC_51_RoHS_P_0.pdf" H 3000 1800 50  0001 C CNN
 F 4 "RESS-018" V 3000 1800 60  0001 C CNN "part_num"
+F 5 "C22859" V 3000 1800 50  0001 C CNN "LCSC"
 	1    3000 1800
 	0    1    1    0
@@
 F 3 "http://www.yageo.com/NewPortal/yageodocoutput?fileName=/pdf/R-Chip/PYu-RC_51_RoHS_P_0.pdf" H 3000 1700 50  0001 C CNN
 F 4 "RESS-018" V 3000 1700 60  0001 C CNN "part_num"
+F 5 "C22859" V 3000 1700 50  0001 C CNN "LCSC"
 	1    3000 1700
 	0    1    1    0
@@
 F 3 "http://www.yageo.com/documents/recent/PYu-RC_Group_51_RoHS_L_10.pdf" H 3000 2350 50  0001 C CNN
 F 4 "RESS-017" V 3000 2350 60  0001 C CNN "part_num"
+F 5 "C21190" V 3000 2350 50  0001 C CNN "LCSC"
 	1    3000 2350
 	0    1    1    0
@@
 F 3 "http://www.yageo.com/documents/recent/PYu-RC_Group_51_RoHS_L_10.pdf" H 2800 2650 50  0001 C CNN
 F 4 "RESS-016" V 2800 2650 60  0001 C CNN "part_num"
+F 5 "C22790" V 2800 2650 50  0001 C CNN "LCSC"
 	1    2800 2650
 	1    0    0    -1
@@
 F 3 "http://industrial.panasonic.com/www-cgi/jvcr13pz.cgi?E+PZ+3+AOA0001+ERJ3GEYJ103V+7+WW" H 2550 2650 50  0001 C CNN
 F 4 "RESS-005" V 2550 2650 60  0001 C CNN "part_num"
+F 5 " C25804" V 2550 2650 50  0001 C CNN "LCSC"
 	1    2550 2650
 	1    0    0    -1
@@
 F 3 "http://www.yageo.com/documents/recent/PYu-RC_Group_51_RoHS_L_10.pdf" H 2550 2050 50  0001 C CNN
 F 4 "RESS-015" V 2550 2050 60  0001 C CNN "part_num"
+F 5 "C23162" V 2550 2050 50  0001 C CNN "LCSC"
 	1    2550 2050
 	1    0    0    -1
